File: Fault_leds.kicad_sch (KiCad schematic)
At the start: 37 parts, among them U7 SN74LVC16T245DGGR

Commit message: Finish BOM
Parts:
- C34, C35, C36, C37: Cost (none) -> .08; MFG (none) -> Taiyo-Yuden; MFG_PN (none) -> TMF212B7104KGHT
- R11, R12, R13, R14, R15, R16, R17, R18, R19, R20, R21, R22, R23, R24, R25, R26: MFG_PN ERJ-2RKF1001X -> ERJ-6ENF6800V
- U7: Cost (none) -> 2.29; MFG Texas Instruments -> TI

Commit message: Nightly commit
Parts:
- C34, C35, C36, C37: footprint Capacitor_SMD:C_0805_2012Metric -> My Footprints:C_0805_2012Metric
Changed lines of the file:
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@@
 			)
 		)
-		(property "Footprint" "Capacitor_SMD:C_0805_2012Metric"
+		(property "Footprint" "My Footprints:C_0805_2012Metric"
 			(at 172.72 52.07 0)
 			(effects
@@
 			)
 		)
-		(property "Footprint" "Capacitor_SMD:C_0805_2012Metric"
+		(property "Footprint" "My Footprints:C_0805_2012Metric"
 			(at 181.61 52.07 0)
 			(effects
@@
 			)
 		)
-		(property "Footprint" "Capacitor_SMD:C_0805_2012Metric"
+		(property "Footprint" "My Footprints:C_0805_2012Metric"
 			(at 95.25 52.07 0)
 			(effects
@@
 			)
 		)
-		(property "Footprint" "Capacitor_SMD:C_0805_2012Metric"
+		(property "Footprint" "My Footprints:C_0805_2012Metric"
 			(at 85.09 52.07 0)
 			(effects
