File: acmi2-afe.kicad_pcb (KiCad board)
At the start: 6 copper layers, 241.3 x 76.2 mm, 130 parts, among them J1 6469028-1, J2 6469028-1, J3 6469028-1, J4 132134, J5 5499922-4, J6 39301022, J7 5499922-4, Q1 NX7002BKW, T1 T1-1T-KK81, U1 200MHz, U10 TPS3850H50DRCR, U2 LTC2107CUK-PBF, U3 TPS7A8500RGRT, U4 TPSM82866AA0HRDMR, U5 TPS7A8500RGRT, U6 TPS259540DSGR, U7 SN74LVC16T245DGGR, U8 CAT25320VI-GT3

Commit message: Nightly commit
Parts:
- C1, C10, C11, C12, C13, C14, C15, C16, C17, C18, C19, C2, C20, C21, C22, C23, C24, C25, C26, C27, C28, C29, C3, C30, C31, C32, C33, C34, C35, C36, C37, C38, C39, C4, C40, C44, C45, C46, C5, C6, C7, C8, C9: footprint Capacitor_SMD:C_0805_2012Metric -> My Footprints:C_0805_2012Metric
- MT1, MT2, MT3, MT4, MT5, MT6, MT7, MT8: footprint MountingHole:MountingHole_4.3mm_M4_DIN965_Pad -> My Footprints:MountingHole_4.3mm_M4_DIN965_Pad
Routing:
- net GND: track 204.5 -> 206.7 mm
- net +3.3V: track 28.0 -> 30.0 mm
- net +5.0V: track 36.9 -> 37.4 mm
