File: adc.kicad_sch (KiCad schematic)
At the start: 21 parts, among them J4 Conn_Coaxial, T1 T1-1T-KK81, U1 200MHz, U2 LTC2107CUK-PBF

Commit message: Finish routing
Parts:
- added C40: 0.1u, Capacitor_SMD:C_0805_2012Metric, symbol Device:C_Small
Connections:
- net GND: now also C40.1; no longer T1.6
- net AIN_P: now reaches R4.1, R6.2
- net AIN_P: now also U2.8 (AIN+); no longer U2.9 (AIN-)
- net AIN_N: now reaches R3.1, R6.1
- net AIN_N: now also U2.9 (AIN-); no longer U2.8 (AIN+)
- net at T1.4: now also C40.2; no longer C2.2
- net adc_clk_n renamed ADC_CLK_N
- net ADC_CLK_N: now also U2.14 (ENC+); no longer U2.15 (ENC-)
- net adc_clk_p renamed ADC_CLK_P
- net ADC_CLK_P: now also U2.15 (ENC-); no longer U2.14 (ENC+)
- new net: C2.2, T1.6
Other:
- moved on the sheet: C2, J4

Commit message: Finish BOM
Parts:
- C1: value 10p -> 0.1u; Cost (none) -> .08; MFG (none) -> Taiyo-Yuden; MFG_PN (none) -> TMF212B7104KGHT
- C10, C2, C3, C4, C40, C6, C9: Cost (none) -> .08; MFG (none) -> Taiyo-Yuden; MFG_PN (none) -> TMF212B7104KGHT
- C11, C8: Cost (none) -> 0.06; MFG (none) -> Murata; MFG_PN (none) -> GRM21BR61C106KE15K
- C5: Cost (none) -> .49; MFG (none) -> Taiyo-Yuden; MFG_PN (none) -> QVS212CG100JDHT
- C7: Cost (none) -> 0.13; MFG (none) -> Taiyo-Yuden; MFG_PN (none) -> UMK212BB7225KG-T
- J4: value Conn_Coaxial -> 132134; Cost (none) -> 5.5; MFG (none) -> Amphenol; MFG_PN (none) -> 132134
- R1, R2: MFG (none) -> Panasonic; MFG_PN (none) -> ERJ-6ENF31R6V
- R3, R4: MFG_PN (none) -> ERJ-6ENF20R0V
- R5: Cost (none) -> .03; MFG (none) -> Panasonic; MFG_PN (none) -> ERJ-6ENF10R0V
- R6: MFG (none) -> Panasonic; MFG_PN (none) -> ERJ-6ENF2000V
- T1: Cost (none) -> 6.56; MFG (none) -> MiniCircuits; MFG_PN (none) -> T1-1T-KK81+
- U1: Cost (none) -> 14.19
- U2: Cost (none) -> 261.83; MFG (none) -> Analog Devices; MFG_PN (none) -> LTC2107CUK#PBF

Commit message: Nightly commit
Parts:
- C1, C10, C11, C2, C3, C4, C40, C5, C6, C7, C8, C9: footprint Capacitor_SMD:C_0805_2012Metric -> My Footprints:C_0805_2012Metric
Changed lines of the file:
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@@
 			)
 		)
-		(property "Footprint" "Capacitor_SMD:C_0805_2012Metric"
+		(property "Footprint" "My Footprints:C_0805_2012Metric"
 			(at 80.01 171.45 0)
 			(effects
@@
 			)
 		)
-		(property "Footprint" "Capacitor_SMD:C_0805_2012Metric"
+		(property "Footprint" "My Footprints:C_0805_2012Metric"
 			(at 133.35 170.18 0)
 			(effects
@@
 			)
 		)
-		(property "Footprint" "Capacitor_SMD:C_0805_2012Metric"
+		(property "Footprint" "My Footprints:C_0805_2012Metric"
 			(at 271.78 60.96 0)
 			(effects
@@
 			)
 		)
-		(property "Footprint" "Capacitor_SMD:C_0805_2012Metric"
+		(property "Footprint" "My Footprints:C_0805_2012Metric"
 			(at 82.55 111.76 0)
 			(effects
@@
 			)
 		)
-		(property "Footprint" "Capacitor_SMD:C_0805_2012Metric"
+		(property "Footprint" "My Footprints:C_0805_2012Metric"
 			(at 133.35 166.37 0)
 			(effects
@@
 			)
 		)
-		(property "Footprint" "Capacitor_SMD:C_0805_2012Metric"
+		(property "Footprint" "My Footprints:C_0805_2012Metric"
 			(at 208.28 60.96 0)
 			(effects
@@
 			)
 		)
-		(property "Footprint" "Capacitor_SMD:C_0805_2012Metric"
+		(property "Footprint" "My Footprints:C_0805_2012Metric"
 			(at 200.66 90.17 0)
 			(effects
@@
 			)
 		)
-		(property "Footprint" "Capacitor_SMD:C_0805_2012Metric"
+		(property "Footprint" "My Footprints:C_0805_2012Metric"
 			(at 176.53 90.17 0)
 			(effects
@@
 			)
 		)
-		(property "Footprint" "Capacitor_SMD:C_0805_2012Metric"
+		(property "Footprint" "My Footprints:C_0805_2012Metric"
 			(at 170.18 116.84 0)
 			(effects
@@
 			)
 		)
-		(property "Footprint" "Capacitor_SMD:C_0805_2012Metric"
+		(property "Footprint" "My Footprints:C_0805_2012Metric"
 			(at 218.44 60.96 0)
 			(effects
@@
 			)
 		)
-		(property "Footprint" "Capacitor_SMD:C_0805_2012Metric"
+		(property "Footprint" "My Footprints:C_0805_2012Metric"
 			(at 82.55 121.92 0)
 			(effects
@@
 			)
 		)
-		(property "Footprint" "Capacitor_SMD:C_0805_2012Metric"
+		(property "Footprint" "My Footprints:C_0805_2012Metric"
 			(at 261.62 60.96 0)
 			(effects
