File: regulator.kicad_sch (KiCad schematic)
At the start: 37 parts, among them J6 39301022, Q1 NX7002BKW, U3 TPS7A8500RGRT, U4 TPSM82866AA0HRDMR, U5 TPS7A8500RGRT, U6 TPS259540DSGR

Commit message: Finish routing
Connections:
- net +3.3v_U5: now reaches C21.1, C22.1, L2.1, U5.14 (EN), U5.15 (IN), U5.16 (IN), U5.17 (IN)
- net +3.3v_U3: now reaches C12.1, C13.1, L1.1, U3.14 (EN), U3.15 (IN), U3.16 (IN), U3.17 (IN)
- net +5VIN: now reaches J6.2, U6.3 (IN), U6.4 (IN)
Changed lines of the file:
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@@
+		)
+	)
+	(label "+3.3v_U5"
+		(at 173.99 128.27 0)
+		(effects
+			(font
+				(size 1.27 1.27)
+			)
+			(justify left bottom)
+		)
+	)
+	(label "+3.3v_U3"
+		(at 44.45 128.27 0)
+		(effects
+			(font
+				(size 1.27 1.27)
+			)
+			(justify left bottom)
+		)
+	)
+	(label "+5VIN"
+		(at 57.15 33.02 0)
+		(effects
+			(font
+				(size 1.27 1.27)
+			)
+			(justify left bottom)
 		)
 	)

Commit message: Finish BOM
Parts:
- C12, C17, C19, C20, C21, C24, C25, C27, C30: Cost (none) -> 0.35; MFG (none) -> TDK; MFG_PN (none) -> C2012X5R1A476M125AC
- C13, C14, C22, C23, C31, C32, C38: Cost (none) -> .08; MFG (none) -> Taiyo-Yuden; MFG_PN (none) -> TMF212B7104KGHT
- C15, C26: Cost (none) -> 0.11; MFG (none) -> Taiyo-Yuden; MFG_PN (none) -> MAASU21GSL8103MTNA01
- C16, C18, C28, C29: Cost (none) -> 0.06; MFG (none) -> Murata; MFG_PN (none) -> GRM21BR61C106KE15K
- C33: Cost (none) -> .15; MFG (none) -> Kemet; MFG_PN (none) -> C0805X332K5RECTU
- J6: Cost (none) -> 1.67; MFG (none) -> Molex; MFG_PN (none) -> 0039301022
- L1, L2: Cost (none) -> .11; MFG (none) -> Taiyo-Yuden; MFG_PN (none) -> LSMGG160808T331RG
- Q1: Cost 0.1 -> 0.18
- R27: MFG_PN ERJ-2RKF1001X -> ERJ-P06F1001V
- R7: MFG (none) -> Panasonic; MFG_PN (none) -> ERJ-6ENF2053V
- R8: MFG (none) -> Panasonic; MFG_PN (none) -> ERJ-6ENF4700V
- R9: ${DNP} (none) -> ${DNP}; Cost (none) -> 0.01; MFG (none) -> Panasonic; MFG_PN (none) -> ERJ-2RKF1001X
- U3, U5: Cost (none) -> 6.33; MFG Texas Instruments -> TI
- U4: Cost (none) -> 5.14; MFG (none) -> TI; MFG_PN (none) -> TPSM82866AA0HRDMR
- U6: Cost (none) -> 0.74; MFG Texas Instruments -> TI

Commit message: Nightly commit
Parts:
- C12, C13, C14, C15, C16, C17, C18, C19, C20, C21, C22, C23, C24, C25, C26, C27, C28, C29, C30, C31, C32, C33, C38: footprint Capacitor_SMD:C_0805_2012Metric -> My Footprints:C_0805_2012Metric
Changed lines of the file:
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@@
 			)
 		)
-		(property "Footprint" "Capacitor_SMD:C_0805_2012Metric"
+		(property "Footprint" "My Footprints:C_0805_2012Metric"
 			(at 49.53 133.35 0)
 			(effects
@@
 			)
 		)
-		(property "Footprint" "Capacitor_SMD:C_0805_2012Metric"
+		(property "Footprint" "My Footprints:C_0805_2012Metric"
 			(at 133.35 48.26 0)
 			(effects
@@
 			)
 		)
-		(property "Footprint" "Capacitor_SMD:C_0805_2012Metric"
+		(property "Footprint" "My Footprints:C_0805_2012Metric"
 			(at 123.19 48.26 0)
 			(effects
@@
 			)
 		)
-		(property "Footprint" "Capacitor_SMD:C_0805_2012Metric"
+		(property "Footprint" "My Footprints:C_0805_2012Metric"
 			(at 55.88 60.96 0)
 			(effects
@@
 			)
 		)
-		(property "Footprint" "Capacitor_SMD:C_0805_2012Metric"
+		(property "Footprint" "My Footprints:C_0805_2012Metric"
 			(at 179.07 133.35 0)
 			(effects
@@
 			)
 		)
-		(property "Footprint" "Capacitor_SMD:C_0805_2012Metric"
+		(property "Footprint" "My Footprints:C_0805_2012Metric"
 			(at 229.87 48.26 0)
 			(effects
@@
 			)
 		)
-		(property "Footprint" "Capacitor_SMD:C_0805_2012Metric"
+		(property "Footprint" "My Footprints:C_0805_2012Metric"
 			(at 254 134.62 0)
 			(effects
@@
 			)
 		)
-		(property "Footprint" "Capacitor_SMD:C_0805_2012Metric"
+		(property "Footprint" "My Footprints:C_0805_2012Metric"
 			(at 219.71 48.26 0)
 			(effects
@@
 			)
 		)
-		(property "Footprint" "Capacitor_SMD:C_0805_2012Metric"
+		(property "Footprint" "My Footprints:C_0805_2012Metric"
 			(at 40.64 133.35 0)
 			(effects
@@
 			)
 		)
-		(property "Footprint" "Capacitor_SMD:C_0805_2012Metric"
+		(property "Footprint" "My Footprints:C_0805_2012Metric"
 			(at 113.03 48.26 0)
 			(effects
@@
 			)
 		)
-		(property "Footprint" "Capacitor_SMD:C_0805_2012Metric"
+		(property "Footprint" "My Footprints:C_0805_2012Metric"
 			(at 233.68 146.05 0)
 			(effects
@@
 			)
 		)
-		(property "Footprint" "Capacitor_SMD:C_0805_2012Metric"
+		(property "Footprint" "My Footprints:C_0805_2012Metric"
 			(at 133.35 134.62 0)
 			(effects
@@
 			)
 		)
-		(property "Footprint" "Capacitor_SMD:C_0805_2012Metric"
+		(property "Footprint" "My Footprints:C_0805_2012Metric"
 			(at 102.87 146.05 0)
 			(effects
@@
 			)
 		)
-		(property "Footprint" "Capacitor_SMD:C_0805_2012Metric"
+		(property "Footprint" "My Footprints:C_0805_2012Metric"
 			(at 123.19 134.62 0)
 			(effects
@@
 			)
 		)
-		(property "Footprint" "Capacitor_SMD:C_0805_2012Metric"
+		(property "Footprint" "My Footprints:C_0805_2012Metric"
 			(at 21.59 133.35 0)
 			(effects
@@
 			)
 		)
-		(property "Footprint" "Capacitor_SMD:C_0805_2012Metric"
+		(property "Footprint" "My Footprints:C_0805_2012Metric"
 			(at 151.13 133.35 0)
 			(effects
@@
 			)
 		)
-		(property "Footprint" "Capacitor_SMD:C_0805_2012Metric"
+		(property "Footprint" "My Footprints:C_0805_2012Metric"
 			(at 43.18 156.21 0)
 			(effects
@@
 			)
 		)
-		(property "Footprint" "Capacitor_SMD:C_0805_2012Metric"
+		(property "Footprint" "My Footprints:C_0805_2012Metric"
 			(at 243.84 134.62 0)
 			(effects
@@
 			)
 		)
-		(property "Footprint" "Capacitor_SMD:C_0805_2012Metric"
+		(property "Footprint" "My Footprints:C_0805_2012Metric"
 			(at 170.18 133.35 0)
 			(effects
@@
 			)
 		)
-		(property "Footprint" "Capacitor_SMD:C_0805_2012Metric"
+		(property "Footprint" "My Footprints:C_0805_2012Metric"
 			(at 264.16 134.62 0)
 			(effects
@@
 			)
 		)
-		(property "Footprint" "Capacitor_SMD:C_0805_2012Metric"
+		(property "Footprint" "My Footprints:C_0805_2012Metric"
 			(at 113.03 134.62 0)
 			(effects
@@
 			)
 		)
-		(property "Footprint" "Capacitor_SMD:C_0805_2012Metric"
+		(property "Footprint" "My Footprints:C_0805_2012Metric"
 			(at 240.03 48.26 0)
 			(effects
@@
 			)
 		)
-		(property "Footprint" "Capacitor_SMD:C_0805_2012Metric"
+		(property "Footprint" "My Footprints:C_0805_2012Metric"
 			(at 173.99 156.21 0)
 			(effects
